Commit message: Renamed the movable joints to be understandable

File: crane_plus_simulation/urdf/simulated_crane_plus.urdf (robot description, URDF)
Before this commit: robot crane_plus_arm, 20 links, 19 joints
Links:
- removed link crane_plus_lower_arm_bracket_link
- removed link crane_plus_moving_finger_bracket_link
- removed link crane_plus_shoulder_bracket_rev_link
- removed link crane_plus_upper_arm_servo_link
- removed link crane_plus_wrist_bracket_link
- added link gripper_link, mass 0.001; collision box size=0.025 0.0485 0.0375; visual mesh filename=package://crane_plus_description/meshes/f2.stl scale=0.001 0.001 0.001
- added link lower_arm_link, mass 0.001; collision box size=0.028 0.0485 0.065; visual mesh filename=package://crane_plus_description/meshes/f4.stl scale=0.001 0.001 0.001
- added link shoulder_link, mass 0.001; collision box size=0.025 0.0485 0.0375; visual mesh filename=package://crane_plus_description/meshes/f2.stl scale=0.001 0.001 0.001
- added link upper_arm_link, mass 0.001; collision box size=0.05 0.032 0.038; visual mesh filename=package://crane_plus_description/meshes/ax12_box.stl scale=0.001 0.001 0.001
- added link wrist_link, mass 0.001; collision box size=0.025 0.0485 0.0375; visual mesh filename=package://crane_plus_description/meshes/f2.stl scale=0.001 0.001 0.001
Joints:
- removed joint crane_plus_lower_arm_bracket_joint
- removed joint crane_plus_moving_finger_bracket_joint
- removed joint crane_plus_shoulder_bracket_rev_joint
- removed joint crane_plus_upper_arm_servo_joint
- removed joint crane_plus_wrist_bracket_joint
- added joint gripper_joint: type revolute, parent crane_plus_gripper_servo_link, child gripper_link, origin xyz=-0.012 0 0 rpy=-1.570795 0 -1.570795, axis 0 -1 0, limit lower=-2.617 upper=2.617 effort=30 velocity=1.571
- added joint lower_arm_joint: type revolute, parent crane_plus_lower_arm_servo_link, child lower_arm_link, origin xyz=-0.012 0 0 rpy=1.570795 0 1.570795, axis 0 1 0, limit lower=-2.617 upper=2.617 effort=30 velocity=1.571
- added joint shoulder_joint: type revolute, parent crane_plus_shoulder_servo_link, child shoulder_link, origin xyz=-0.0135 0 0.021 rpy=0 0 0, axis 0 0 1, limit lower=-2.617 upper=2.617 effort=30 velocity=1.571
- added joint upper_arm_joint: type revolute, parent shoulder_link, child upper_arm_link, origin xyz=0 0 0.0265 rpy=-1.570795 -1.570795 0, axis 0 0 -1, limit lower=-2.617 upper=2.617 effort=30 velocity=1.571
- added joint wrist_joint: type revolute, parent crane_plus_wrist_servo_link, child wrist_link, origin xyz=-0.012 0 0 rpy=-1.570795 0 -1.570795, axis 0 -1 0, limit lower=-2.617 upper=2.617 effort=30 velocity=1.571
- joint crane_plus_lower_arm_joiner_joint: parent crane_plus_lower_arm_bracket_link -> lower_arm_link
- joint crane_plus_moving_finger_joint: parent crane_plus_moving_finger_bracket_link -> gripper_link
- joint crane_plus_upper_arm_upper_joiner_joint: parent crane_plus_upper_arm_servo_link -> upper_arm_link
- joint crane_plus_wrist_joiner_joint: parent crane_plus_wrist_bracket_link -> wrist_link

File: crane_plus_simulation/urdf/simulated_crane_plus.urdf.xacro (robot description, xacro)
@@ -25,5 +25,5 @@
   <transmission name="shoulder">
     <type>transmission_interface/SimpleTransmission</type>
-    <joint name="crane_plus_shoulder_bracket_rev_joint">
+    <joint name="shoulder_joint">
       <hardwareInterface>PositionJointInterface</hardwareInterface>
     </joint>
@@ -36,5 +36,5 @@
   <transmission name="upper_arm">
     <type>transmission_interface/SimpleTransmission</type>
-    <joint name="crane_plus_upper_arm_servo_joint">
+    <joint name="upper_arm_joint">
       <hardwareInterface>PositionJointInterface</hardwareInterface>
     </joint>
@@ -47,5 +47,5 @@
   <transmission name="lower_arm">
     <type>transmission_interface/SimpleTransmission</type>
-    <joint name="crane_plus_lower_arm_bracket_joint">
+    <joint name="lower_arm_joint">
       <hardwareInterface>PositionJointInterface</hardwareInterface>
     </joint>
@@ -58,5 +58,5 @@
   <transmission name="wrist">
     <type>transmission_interface/SimpleTransmission</type>
-    <joint name="crane_plus_wrist_bracket_joint">
+    <joint name="wrist_joint">
       <hardwareInterface>PositionJointInterface</hardwareInterface>
     </joint>
@@ -69,5 +69,5 @@
   <transmission name="gripper">
     <type>transmission_interface/SimpleTransmission</type>
-    <joint name="crane_plus_moving_finger_bracket_joint">
+    <joint name="gripper_joint">
       <hardwareInterface>PositionJointInterface</hardwareInterface>
     </joint>
@@ -81,9 +81,9 @@
     <plugin name="joint_state_publisher" filename="libgazebo_ros_joint_state_publisher.so">
       <jointName>
-        crane_plus_shoulder_bracket_rev_joint,
-        crane_plus_upper_arm_servo_joint,
-        crane_plus_lower_arm_bracket_joint,
-        crane_plus_wrist_bracket_joint,
-        crane_plus_moving_finger_bracket_joint
+        shoulder_joint,
+        upper_arm_joint,
+        lower_arm_joint,
+        wrist_joint,
+        gripper_joint
       </jointName>
     </plugin>
