Commit message: Make simulator use the same parent frame as hardware

File: crane_plus_simulation/urdf/simulated_crane_plus.urdf.xacro (robot description, xacro)
@@ -9,10 +9,10 @@
   <xacro:include filename="$(find crane_plus_description)/urdf/crane_plus.xacro"/>
   <!-- Link to provide the location reference for the arm -->
-  <link name="world"/>
+  <link name="base_link"/>
   <!-- Use the crane_plus macro to configure a Crane+ arm with desired joint
        velocities limit and lower/upper limits for the first joint. This
        allows accessing different operational areas, e.g. left-handed vs.
        right-handed robots. -->
-  <crane_plus parent="world"
+  <crane_plus parent="base_link"
               servo_color="black" bracket_color="grey" gripper_color="black"
               joints_vlimit="1.571"
