Commit message: Working on arm model

File: crane_plus_description/urdf/crane_plus.urdf (robot description, URDF)
Before this commit: robot crane_plus, 6 links, 5 joints
Links:
- removed link link1
- removed link link2
- removed link link3
- removed link link4
- removed link link5
- added link crane_plus_base_bracket_link, mass 0.00001; collision box size=0.022 0.032 0.007; visual mesh filename=package://crane_plus_description/meshes/f53.stl scale=0.01 0.01 0.01
- added link crane_plus_base_link
- added link crane_plus_mounting_plate_link, mass 0.00001; collision box size=0.05 0.05 0.001; visual mesh filename=package://crane_plus_description/meshes/mount.stl scale=1 1 1
- added link crane_plus_shoulder_bracket_rev_link, mass 0.00001; collision box size=0.025 0.0485 0.0375; visual mesh filename=package://crane_plus_description/meshes/f2.stl scale=0.001 0.001 0.001
- added link crane_plus_shoulder_servo_link, mass 0.00001; collision box size=0.05 0.032 0.038; visual mesh filename=package://crane_plus_description/meshes/ax12_box.stl scale=0.001 0.001 0.001
- link base_link: geometry 
Joints:
- removed joint joint1
- removed joint joint2
- removed joint joint3
- removed joint joint4
- removed joint joint5
- added joint crane_plus_base_bracket_joint: type fixed, parent crane_plus_mounting_plate_link, child crane_plus_base_bracket_link, origin xyz=0 0 0.001 rpy=0 0 0
- added joint crane_plus_base_joint: type fixed, parent base_link, child crane_plus_base_link, origin xyz=0 0 0
- added joint crane_plus_mounting_plate_joint: type fixed, parent crane_plus_base_link, child crane_plus_mounting_plate_link, origin xyz=0 0 0 rpy=0 0 0
- added joint crane_plus_shoulder_bracket_rev_joint: type revolute, parent crane_plus_shoulder_servo_link, child crane_plus_shoulder_bracket_rev_link, origin xyz=-0.0135 0 0.04 rpy=0 0 0, axis 0 0 1, limit lower=-2.617 upper=2.617 effort=30 velocity=1.571
- added joint crane_plus_shoulder_servo_joint: type fixed, parent crane_plus_base_bracket_link, child crane_plus_shoulder_servo_link, origin xyz=0 0 0.004 rpy=0 0 0

Commit message: Finished visual and collision models

File: crane_plus_description/urdf/crane_plus.urdf (robot description, URDF)
Before this commit: robot crane_plus_arm, 6 links, 5 joints
Links:
- added link crane_plus_fixed_finger_joiner_link, mass 0.00001; collision box size=0.025 0.038 0.009; visual mesh filename=package://crane_plus_description/meshes/f3.stl scale=0.001 0.001 0.001
- added link crane_plus_fixed_finger_link, mass 0.00001; collision mesh filename=package://crane_plus_description/meshes/finger_fixed_collis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 scale=0.001 0.001 0.001; visual mesh filename=package://crane_plus_description/meshes/finger_fixed.stl scale=0.001 0.001 0.001
- added link crane_plus_gripper_servo_link, mass 0.00001; collision box size=0.05 0.032 0.038; visual mesh filename=package://crane_plus_description/meshes/ax12_box.stl scale=0.001 0.001 0.001
- added link crane_plus_lower_arm_bracket_link, mass 0.00001; collision box size=0.028 0.0485 0.065; visual mesh filename=package://crane_plus_description/meshes/f4.stl scale=0.001 0.001 0.001
- added link crane_plus_lower_arm_joiner_link, mass 0.00001; collision box size=0.025 0.038 0.009; visual mesh filename=package://crane_plus_description/meshes/f3.stl scale=0.001 0.001 0.001
- added link crane_plus_lower_arm_servo_link, mass 0.00001; collision box size=0.05 0.032 0.038; visual mesh filename=package://crane_plus_description/meshes/ax12_box.stl scale=0.001 0.001 0.001
- added link crane_plus_moving_finger_bracket_link, mass 0.00001; collision box size=0.025 0.0485 0.0375; visual mesh filename=package://crane_plus_description/meshes/f2.stl scale=0.001 0.001 0.001
- added link crane_plus_moving_finger_link, mass 0.00001; collision mesh filename=package://crane_plus_description/meshes/finger_moving_colli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 scale=0.001 0.001 0.001; visual mesh filename=package://crane_plus_description/meshes/finger_moving.stl scale=0.001 0.001 0.001
- added link crane_plus_upper_arm_lower_joiner_link, mass 0.00001; collision box size=0.025 0.038 0.009; visual mesh filename=package://crane_plus_description/meshes/f3.stl scale=0.001 0.001 0.001
- added link crane_plus_upper_arm_servo_link, mass 0.00001; collision box size=0.05 0.032 0.038; visual mesh filename=package://crane_plus_description/meshes/ax12_box.stl scale=0.001 0.001 0.001
- added link crane_plus_upper_arm_upper_joiner_link, mass 0.00001; collision box size=0.025 0.038 0.009; visual mesh filename=package://crane_plus_description/meshes/f3.stl scale=0.001 0.001 0.001
- added link crane_plus_wrist_bracket_link, mass 0.00001; collision box size=0.025 0.0485 0.0375; visual mesh filename=package://crane_plus_description/meshes/f2.stl scale=0.001 0.001 0.001
- added link crane_plus_wrist_joiner_link, mass 0.00001; collision box size=0.025 0.038 0.009; visual mesh filename=package://crane_plus_description/meshes/f3.stl scale=0.001 0.001 0.001
- added link crane_plus_wrist_servo_link, mass 0.00001; collision box size=0.05 0.032 0.038; visual mesh filename=package://crane_plus_description/meshes/ax12_box.stl scale=0.001 0.001 0.001
- link crane_plus_base_bracket_link: geometry collision box size=0.022 0.032 0.008; visual mesh filename=package://crane_plus_description/meshes/f53.stl scale=0.01 0.01 0.01
Joints:
- added joint crane_plus_fixed_finger_joiner_joint: type fixed, parent crane_plus_gripper_servo_link, child crane_plus_fixed_finger_joiner_link, origin xyz=0.0295 0 0 rpy=-1.570795 0 1.570795
- added joint crane_plus_fixed_finger_joint: type fixed, parent crane_plus_fixed_finger_joiner_link, child crane_plus_fixed_finger_link, origin xyz=0 0 0 rpy=0 0 3.14159
- added joint crane_plus_gripper_servo_joint: type fixed, parent crane_plus_wrist_joiner_link, child crane_plus_gripper_servo_link, origin xyz=0.0028 0 0.019 rpy=1.570795 3.14159 0
- added joint crane_plus_lower_arm_bracket_joint: type revolute, parent crane_plus_lower_arm_servo_link, child crane_plus_lower_arm_bracket_link, origin xyz=-0.012 0 0 rpy=1.570795 0 1.570795, axis 0 1 0, limit lower=-2.617 upper=2.617 effort=30 velocity=1.571
- added joint crane_plus_lower_arm_joiner_joint: type fixed, parent crane_plus_lower_arm_bracket_link, child crane_plus_lower_arm_joiner_link, origin xyz=0 0 -0.0525 rpy=0 3.14159 0
- added joint crane_plus_lower_arm_servo_joint: type fixed, parent crane_plus_upper_arm_lower_joiner_link, child crane_plus_lower_arm_servo_link, origin xyz=0 0 0.0295 rpy=0 1.570795 1.570795
- added joint crane_plus_moving_finger_bracket_joint: type revolute, parent crane_plus_gripper_servo_link, child crane_plus_moving_finger_bracket_link, origin xyz=-0.012 0 0 rpy=-1.570795 0 -1.570795, axis 0 1 0, limit lower=-2.617 upper=2.617 effort=30 velocity=1.571
- added joint crane_plus_moving_finger_joint: type fixed, parent crane_plus_moving_finger_bracket_link, child crane_plus_moving_finger_link, origin xyz=0 0 -0.0265 rpy=3.14159 0 0
- added joint crane_plus_upper_arm_lower_joiner_joint: type fixed, parent crane_plus_upper_arm_upper_joiner_link, child crane_plus_upper_arm_lower_joiner_link, origin xyz=0 0 0 rpy=3.14159 0 0
- added joint crane_plus_upper_arm_servo_joint: type revolute, parent crane_plus_shoulder_bracket_rev_link, child crane_plus_upper_arm_servo_link, origin xyz=0 0 0.0265 rpy=-1.570795 -1.570795 0, axis 0 0 1, limit lower=-2.617 upper=2.617 effort=30 velocity=1.571
- added joint crane_plus_upper_arm_upper_joiner_joint: type fixed, parent crane_plus_upper_arm_servo_link, child crane_plus_upper_arm_upper_joiner_link, origin xyz=0.0415 0 0 rpy=-1.570795 0 1.570795
- added joint crane_plus_wrist_bracket_joint: type revolute, parent crane_plus_wrist_servo_link, child crane_plus_wrist_bracket_link, origin xyz=-0.012 0 0 rpy=-1.570795 0 -1.570795, axis 0 1 0, limit lower=-2.617 upper=2.617 effort=30 velocity=1.571
- added joint crane_plus_wrist_joiner_joint: type fixed, parent crane_plus_wrist_bracket_link, child crane_plus_wrist_joiner_link, origin xyz=0 0 -0.0265 rpy=0 3.14159 1.570795
- added joint crane_plus_wrist_servo_joint: type fixed, parent crane_plus_lower_arm_joiner_link, child crane_plus_wrist_servo_link, origin xyz=0 0 0.0295 rpy=0 1.570795 1.570795
- joint crane_plus_shoulder_bracket_rev_joint: origin xyz=-0.0135 0 0.04 rpy=0 0 0 -> xyz=-0.0135 0 0.021 rpy=0 0 0
- joint crane_plus_shoulder_servo_joint: origin xyz=0 0 0.004 rpy=0 0 0 -> xyz=-0.0028 0 0.023 rpy=0 0 0

File: crane_plus_description/urdf/crane_plus.xacro (robot description, xacro)
@@ -35,8 +35,8 @@
         name="crane_plus_shoulder_servo"
         color="black">
-      <origin xyz="0 0 ${F53_HEIGHT}" rpy="0 0 0"/>
+        <origin xyz="-${AX12_SIDE_SCREW_OFFSET} 0 ${AX12_BODY_MAIN_HEIGHT/2 + F53_HEIGHT}" rpy="0 0 0"/>
     </dynamixel_ax12_fixed>
     <!-- Shoulder bracket -->
-    <bioloid_f2_revolute
+    <bioloid_f2_revolute_base_axis
         parent="crane_plus_shoulder_servo_link"
         name="crane_plus_shoulder_bracket_rev"
@@ -45,6 +45,116 @@
         llimit="${pan_llimit}"
         ulimit="${pan_ulimit}">
-      <origin xyz="-${AX12_AXEL_OFFSET} 0 ${AX12_HEIGHT}" rpy="0 0 0"/>
+        <origin xyz="-${AX12_AXLE_OFFSET} 0 ${AX12_HORN_HEIGHT}" rpy="0 0 0"/>
+    </bioloid_f2_revolute_base_axis>
+    <!--Upper arm servo -->
+    <dynamixel_ax12_revolute
+        parent="crane_plus_shoulder_bracket_rev_link"
+        name="crane_plus_upper_arm_servo"
+        color="black"
+        vlimit="${joints_vlimit}"
+        llimit="${pan_llimit}"
+        ulimit="${pan_ulimit}">
+        <origin xyz="0 0 ${F2_AXLE_HEIGHT}" rpy="-${M_PI/2} -${M_PI/2} 0"/>
+    </dynamixel_ax12_revolute>
+    <!-- Upper arm upper joiner -->
+    <bioloid_f3_fixed
+        parent="crane_plus_upper_arm_servo_link"
+        name="crane_plus_upper_arm_upper_joiner"
+        color="grey">
+        <origin xyz="${AX12_ORIGIN_TO_AXLE+AX12_ORIGIN_TO_END_SCREW+F3_SCREW_HEIGHT} 0 0" rpy="-${M_PI/2} 0 ${M_PI/2}"/>
+    </bioloid_f3_fixed>
+    <!-- Upper arm lower joiner -->
+    <bioloid_f3_fixed
+        parent="crane_plus_upper_arm_upper_joiner_link"
+        name="crane_plus_upper_arm_lower_joiner"
+        color="grey">
+        <origin xyz="0 0 0" rpy="${M_PI} 0 0"/>
+    </bioloid_f3_fixed>
+    <!-- Lower arm servo -->
+    <dynamixel_ax12_fixed
+        parent="crane_plus_upper_arm_lower_joiner_link"
+        name="crane_plus_lower_arm_servo"
+        color="black">
+      <origin xyz="0 0 ${F3_SCREW_HEIGHT+AX12_ORIGIN_TO_END_SCREW}" rpy="0 ${M_PI/2} ${M_PI/2}"/>
+    </dynamixel_ax12_fixed>
+    <!-- Lower arm bracket -->
+    <bioloid_f4_revolute
+        parent="crane_plus_lower_arm_servo_link"
+        name="crane_plus_lower_arm_bracket"
+        color="grey"
+        vlimit="${joints_vlimit}"
+        llimit="${pan_llimit}"
+        ulimit="${pan_ulimit}">
+        <origin xyz="-${AX12_ORIGIN_TO_AXLE} 0 0" rpy="${M_PI/2} 0 ${M_PI/2}"/>
+    </bioloid_f4_revolute>
+    <!-- Lower arm joiner -->
+    <bioloid_f3_fixed
+        parent="crane_plus_lower_arm_bracket_link"
+        name="crane_plus_lower_arm_joiner"
+        color="grey">
+        <origin xyz="0 0 -${F4_AXLE_HEIGHT}" rpy="0 ${M_PI} 0"/>
+    </bioloid_f3_fixed>
+    <!-- Wrist servo -->
+    <dynamixel_ax12_fixed
+        parent="crane_plus_lower_arm_joiner_link"
+        name="crane_plus_wrist_servo"
+        color="black">
+      <origin xyz="0 0 ${F3_SCREW_HEIGHT+AX12_ORIGIN_TO_END_SCREW}" rpy="0 ${M_PI/2} ${M_PI/2}"/>
+    </dynamixel_ax12_fixed>
+    <!-- Wrist bracket -->
+    <bioloid_f2_revolute
+        parent="crane_plus_wrist_servo_link"
+        name="crane_plus_wrist_bracket"
+        color="grey"
+        vlimit="${joints_vlimit}"
+        llimit="${pan_llimit}"
+        ulimit="${pan_ulimit}">
+        <origin xyz="-${AX12_ORIGIN_TO_AXLE} 0 0" rpy="-${M_PI/2} 0 -${M_PI/2}"/>
     </bioloid_f2_revolute>
+    <!-- Wrist joiner -->
+    <bioloid_f3_fixed
+        parent="crane_plus_wrist_bracket_link"
+        name="crane_plus_wrist_joiner"
+        color="grey">
+        <origin xyz="0 0 -${F2_AXLE_HEIGHT}" rpy="0 ${M_PI} ${M_PI/2}"/>
+    </bioloid_f3_fixed>
+    <!-- Gripper servo -->
+    <dynamixel_ax12_fixed
+        parent="crane_plus_wrist_joiner_link"
+        name="crane_plus_gripper_servo"
+        color="black">
+        <origin xyz="${AX12_SIDE_SCREW_OFFSET} 0 ${F3_SCREW_HEIGHT+AX12_ORIGIN_TO_SIDE_SCREW}" rpy="${M_PI/2} ${M_PI} 0"/>
+    </dynamixel_ax12_fixed>
+    <!-- Fixed finger joiner -->
+    <bioloid_f3_fixed
+        parent="crane_plus_gripper_servo_link"
+        name="crane_plus_fixed_finger_joiner"
+        color="grey">
+        <origin xyz="${AX12_ORIGIN_TO_END_SCREW+F3_SCREW_HEIGHT} 0 0" rpy="-${M_PI/2} 0 ${M_PI/2}"/>
+    </bioloid_f3_fixed>
+    <!-- Fixed finger -->
+    <fixed_finger
+        parent="crane_plus_fixed_finger_joiner_link"
+        name="crane_plus_fixed_finger"
+        color="black">
+      <origin xyz="0 0 0" rpy="0 0 ${M_PI}"/>
+    </fixed_finger>
+    <!-- Wrist bracket -->
+    <bioloid_f2_revolute
+        parent="crane_plus_gripper_servo_link"
+        name="crane_plus_moving_finger_bracket"
+        color="grey"
+        vlimit="${joints_vlimit}"
+        llimit="${pan_llimit}"
+        ulimit="${pan_ulimit}">
+        <origin xyz="-${AX12_ORIGIN_TO_AXLE} 0 0" rpy="-${M_PI/2} 0 -${M_PI/2}"/>
+    </bioloid_f2_revolute>
+    <!-- Movin finger -->
+    <moving_finger
+        parent="crane_plus_moving_finger_bracket_link"
+        name="crane_plus_moving_finger"
+        color="black">
+      <origin xyz="0 0 -${F2_AXLE_HEIGHT}" rpy="${M_PI} 0 0"/>
+    </moving_finger>
   </xacro:macro>
 </robot>
