Commit message: Add MoveIt! configuration package

File: crane_plus_description/urdf/crane_plus.urdf (robot description, URDF)
Before this commit: robot crane_plus_arm, 20 links, 19 joints
Links:
- removed link base_link
- added link world
- link crane_plus_base_bracket_link: mass 0.005 -> 0.001
- link crane_plus_fixed_finger_joiner_link: mass 0.005 -> 0.001
- link crane_plus_fixed_finger_link: mass 0.02 -> 0.001
- link crane_plus_gripper_servo_link: mass 0.0564 -> 0.001
- link crane_plus_lower_arm_bracket_link: mass 0.015 -> 0.001
- link crane_plus_lower_arm_joiner_link: mass 0.005 -> 0.001
- link crane_plus_lower_arm_servo_link: mass 0.0564 -> 0.001
- link crane_plus_mounting_plate_link: mass 0.02 -> 0.001
- link crane_plus_moving_finger_bracket_link: mass 0.01 -> 0.001
- link crane_plus_moving_finger_link: mass 0.02 -> 0.001
- link crane_plus_shoulder_bracket_rev_link: mass 0.01 -> 0.001
- link crane_plus_shoulder_servo_link: mass 0.0564 -> 0.001
- link crane_plus_upper_arm_lower_joiner_link: mass 0.005 -> 0.001
- link crane_plus_upper_arm_servo_link: mass 0.0564 -> 0.001
- link crane_plus_upper_arm_upper_joiner_link: mass 0.005 -> 0.001
- link crane_plus_wrist_bracket_link: mass 0.01 -> 0.001
- link crane_plus_wrist_joiner_link: mass 0.005 -> 0.001
- link crane_plus_wrist_servo_link: mass 0.0564 -> 0.001
Joints:
- joint crane_plus_base_joint: parent base_link -> world

File: crane_plus_description/urdf/crane_plus.urdf.xacro (robot description, xacro)
@@ -9,10 +9,10 @@
   <xacro:include filename="$(find crane_plus_description)/urdf/crane_plus.xacro"/>
   <!-- Link to provide the location reference for the arm -->
-  <link name="base_link"/>
+  <link name="world"/>
   <!-- Use the crane_plus macro to configure a Crane+ arm with desired joint
        velocities limit and lower/upper limits for the first joint. This
        allows accessing different operational areas, e.g. left-handed vs.
        right-handed robots. -->
-  <crane_plus parent="base_link"
+  <crane_plus parent="world"
               servo_color="black" bracket_color="grey" gripper_color="black"
               joints_vlimit="1.571"

File: crane_plus_description/urdf/crane_plus_hardware.xacro (robot description, xacro)
@@ -56,10 +56,17 @@
     </joint>
     <link name="${name}_link">
-      <inertial>
-        <mass value="0.02"/>
-        <origin xyz="0 0 0.0005" rpy="0 0 0"/>
-        <inertia ixx="4.1683e-6" ixy="0.0" ixz="0.0"
-          iyy="8.33e-6" iyz="0.0"
-          izz="4.1683e-6"/>
+      <!--<inertial>-->
+        <!--<mass value="0.02"/>-->
+        <!--<origin xyz="0 0 0.0005" rpy="0 0 0"/>-->
+        <!--<inertia ixx="4.1683e-6" ixy="0.0" ixz="0.0"-->
+          <!--iyy="8.33e-6" iyz="0.0"-->
+          <!--izz="4.1683e-6"/>-->
+      <!--</inertial>-->
+      <inertial>
+        <mass value="0.001"/>
+        <origin xyz="0 0 0.0005" rpy="0 0 0"/>
+        <inertia ixx="1" ixy="0.0" ixz="0.0"
+          iyy="1" iyz="0.0"
+          izz="1"/>
       </inertial>
       <visual>
@@ -86,19 +93,26 @@
     <link name="${name}_link">
       <inertial>
-        <mass value="0.005"/>
+        <mass value="0.001"/>
+        <origin xyz="0 0 0.0005" rpy="0 0 0"/>
+        <inertia ixx="1" ixy="0.0" ixz="0.0"
+          iyy="1" iyz="0.0"
+          izz="1"/>
+      </inertial>
+      <!--<inertial>-->
+        <!--<mass value="0.005"/>-->
+        <!--<origin xyz="0.0 0.0 0.004" rpy="0 0 0"/>-->
+        <!--<inertia ixx="4.53e-7" ixy="0.0" ixz="0.0"-->
+          <!--iyy="6.283e-7" iyz="0.0"-->
+          <!--izz="2.283e-7"/>-->
+      <!--</inertial>-->
+      <visual>
+        <origin xyz="0 0 0" rpy="-${M_PI/2} 0 0"/>
+        <geometry>
+          <mesh filename="package://crane_plus_description/meshes/f53.stl" scale="${SCALE_CM} ${SCALE_CM} ${SCALE_CM}"/>
+        </geometry>
+        <material name="${color}"/>
+      </visual>
+      <collision>
         <origin xyz="0.0 0.0 0.004" rpy="0 0 0"/>
-        <inertia ixx="4.53e-7" ixy="0.0" ixz="0.0"
-          iyy="6.283e-7" iyz="0.0"
-          izz="2.283e-7"/>
-      </inertial>
-      <visual>
-        <origin xyz="0 0 0" rpy="-${M_PI/2} 0 0"/>
-        <geometry>
-          <mesh filename="package://crane_plus_description/meshes/f53.stl" scale="${SCALE_CM} ${SCALE_CM} ${SCALE_CM}"/>
-        </geometry>
-        <material name="${color}"/>
-      </visual>
-      <collision>
-        <origin xyz="0.0 0.0 0.004" rpy="0 0 0"/>
         <geometry>
           <box size="0.022 0.032 0.008"/>
@@ -115,10 +129,17 @@
     <link name="${name}_link">
       <inertial>
-        <mass value="0.0564"/>
-        <origin xyz="${0-AX12_ORIGIN_OFFSET_X} 0 0" rpy="0 0 0"/>
-        <inertia ixx="1.16e-5" ixy="0.0" ixz="0.0"
-          iyy="1.656e-50" iyz="0.0"
-          izz="1.854e-5"/>
-      </inertial>
+        <mass value="0.001"/>
+        <origin xyz="0 0 0.0005" rpy="0 0 0"/>
+        <inertia ixx="1" ixy="0.0" ixz="0.0"
+          iyy="1" iyz="0.0"
+          izz="1"/>
+      </inertial>
+      <!--<inertial>-->
+        <!--<mass value="0.0564"/>-->
+        <!--<origin xyz="${0-AX12_ORIGIN_OFFSET_X} 0 0" rpy="0 0 0"/>-->
+        <!--<inertia ixx="1.16e-5" ixy="0.0" ixz="0.0"-->
+          <!--iyy="1.656e-50" iyz="0.0"-->
+          <!--izz="1.854e-5"/>-->
+      <!--</inertial>-->
       <visual>
         <origin xyz="0 0 0" rpy="-${M_PI/2} 0 0"/>
@@ -146,10 +167,17 @@
     <link name="${name}_link">
       <inertial>
-        <mass value="0.0564"/>
-        <origin xyz="${AX12_ORIGIN_TO_AXLE-AX12_ORIGIN_OFFSET_X} 0 0" rpy="0 0 0"/>
-        <inertia ixx="1.16e-5" ixy="0.0" ixz="0.0"
-          iyy="1.656e-5" iyz="0.0"
-          izz="1.854e-5"/>
-      </inertial>
+        <mass value="0.001"/>
+        <origin xyz="0 0 0.0005" rpy="0 0 0"/>
+        <inertia ixx="1" ixy="0.0" ixz="0.0"
+          iyy="1" iyz="0.0"
+          izz="1"/>
+      </inertial>
+      <!--<inertial>-->
+        <!--<mass value="0.0564"/>-->
+        <!--<origin xyz="${AX12_ORIGIN_TO_AXLE-AX12_ORIGIN_OFFSET_X} 0 0" rpy="0 0 0"/>-->
+        <!--<inertia ixx="1.16e-5" ixy="0.0" ixz="0.0"-->
+          <!--iyy="1.656e-5" iyz="0.0"-->
+          <!--izz="1.854e-5"/>-->
+      <!--</inertial>-->
       <visual>
         <origin xyz="${AX12_ORIGIN_TO_AXLE} 0 0" rpy="-${M_PI/2} 0 0"/>
@@ -177,12 +205,19 @@
     <link name="${name}_link">
       <inertial>
-        <mass value="0.01"/>
-        <origin xyz="0 0 0.01875" rpy="0 0 0"/>
-        <!-- Full height: (3.1320833333333333e-06, 2.481041666666667e-06, 1.6927083333333333e-06) -->
-        <!-- Half height: (2.253177083333333e-06, 2.481041666666667e-06, 8.138020833333333e-07) -->
-        <inertia ixx="2.253e-6" ixy="0.0" ixz="0.0"
-          iyy="2.481e-6" iyz="0.0"
-          izz="8.138e-7"/>
-      </inertial>
+        <mass value="0.001"/>
+        <origin xyz="0 0 0.0005" rpy="0 0 0"/>
+        <inertia ixx="1" ixy="0.0" ixz="0.0"
+          iyy="1" iyz="0.0"
+          izz="1"/>
+      </inertial>
+      <!--<inertial>-->
+        <!--<mass value="0.01"/>-->
+        <!--<origin xyz="0 0 0.01875" rpy="0 0 0"/>-->
+        <!--[> Full height: (3.1320833333333333e-06, 2.481041666666667e-06, 1.6927083333333333e-06) <]-->
+        <!--[> Half height: (2.253177083333333e-06, 2.481041666666667e-06, 8.138020833333333e-07) <]-->
+        <!--<inertia ixx="2.253e-6" ixy="0.0" ixz="0.0"-->
+          <!--iyy="2.481e-6" iyz="0.0"-->
+          <!--izz="8.138e-7"/>-->
+      <!--</inertial>-->
       <visual>
         <origin xyz="0 0 ${F2_AXLE_HEIGHT}" rpy="${M_PI/2} 0 0"/>
@@ -210,21 +245,28 @@
     <link name="${name}_link">
       <inertial>
-        <mass value="0.01"/>
+        <mass value="0.001"/>
+        <origin xyz="0 0 0.0005" rpy="0 0 0"/>
+        <inertia ixx="1" ixy="0.0" ixz="0.0"
+          iyy="1" iyz="0.0"
+          izz="1"/>
+      </inertial>
+      <!--<inertial>-->
+        <!--<mass value="0.01"/>-->
+        <!--<origin xyz="0 0 -${F2_AXLE_HEIGHT-F2_HEIGHT/2}" rpy="0 0 0"/>-->
+        <!--[> Full height: (3.1320833333333333e-06, 2.481041666666667e-06, 1.6927083333333333e-06) <]-->
+        <!--[> Half height: (2.253177083333333e-06, 2.481041666666667e-06, 8.138020833333333e-07) <]-->
+        <!--<inertia ixx="2.253e-6" ixy="0.0" ixz="0.0"-->
+          <!--iyy="2.481e-6" iyz="0.0"-->
+          <!--izz="8.138e-7"/>-->
+      <!--</inertial>-->
+      <visual>
+        <origin xyz="0 0 0" rpy="${M_PI/2} 0 0"/>
+        <geometry>
+          <mesh filename="package://crane_plus_description/meshes/f2.stl" scale="${SCALE_MM} ${SCALE_MM} ${SCALE_MM}"/>
+        </geometry>
+        <material name="${color}"/>
+      </visual>
+      <collision>
         <origin xyz="0 0 -${F2_AXLE_HEIGHT-F2_HEIGHT/2}" rpy="0 0 0"/>
-        <!-- Full height: (3.1320833333333333e-06, 2.481041666666667e-06, 1.6927083333333333e-06) -->
-        <!-- Half height: (2.253177083333333e-06, 2.481041666666667e-06, 8.138020833333333e-07) -->
-        <inertia ixx="2.253e-6" ixy="0.0" ixz="0.0"
-          iyy="2.481e-6" iyz="0.0"
-          izz="8.138e-7"/>
-      </inertial>
-      <visual>
-        <origin xyz="0 0 0" rpy="${M_PI/2} 0 0"/>
-        <geometry>
-          <mesh filename="package://crane_plus_description/meshes/f2.stl" scale="${SCALE_MM} ${SCALE_MM} ${SCALE_MM}"/>
-        </geometry>
-        <material name="${color}"/>
-      </visual>
-      <collision>
-        <origin xyz="0 0 -${F2_AXLE_HEIGHT-F2_HEIGHT/2}" rpy="0 0 0"/>
         <geometry>
           <box size="0.025 0.0485 0.0375"/>
@@ -241,10 +283,17 @@
     <link name="${name}_link">
       <inertial>
-        <mass value="0.005"/>
-        <origin xyz="0.0 0.0 0.0045" rpy="0 0 0"/>
-        <inertia ixx="6.354e-7" ixy="0.0" ixz="0.0"
-          iyy="8.621e-7" iyz="0.0"
-          izz="2.942e-7"/>
-      </inertial>
+        <mass value="0.001"/>
+        <origin xyz="0 0 0.0005" rpy="0 0 0"/>
+        <inertia ixx="1" ixy="0.0" ixz="0.0"
+          iyy="1" iyz="0.0"
+          izz="1"/>
+      </inertial>
+      <!--<inertial>-->
+        <!--<mass value="0.005"/>-->
+        <!--<origin xyz="0.0 0.0 0.0045" rpy="0 0 0"/>-->
+        <!--<inertia ixx="6.354e-7" ixy="0.0" ixz="0.0"-->
+          <!--iyy="8.621e-7" iyz="0.0"-->
+          <!--izz="2.942e-7"/>-->
+      <!--</inertial>-->
       <visual>
         <origin xyz="0 0 0" rpy="${M_PI/2} 0 ${M_PI}"/>
@@ -272,12 +321,19 @@
     <link name="${name}_link">
       <inertial>
-        <mass value="0.015"/>
-        <origin xyz="0 0 -${F4_AXLE_HEIGHT-F4_HEIGHT/2+0.0015}" rpy="0 0 0"/>
-        <!-- Full height: (8.2215625e-06, 3.9203124999999996e-06, 6.2612499999999996e-06) -->
-        <!-- Half height: (4.2606249999999995e-06, 3.9203124999999996e-06, 2.3003125e-06) -->
-        <inertia ixx="4.261e-6" ixy="0.0" ixz="0.0"
-          iyy="3.921e-6" iyz="0.0"
-          izz="2.3e-6"/>
-      </inertial>
+        <mass value="0.001"/>
+        <origin xyz="0 0 0.0005" rpy="0 0 0"/>
+        <inertia ixx="1" ixy="0.0" ixz="0.0"
+          iyy="1" iyz="0.0"
+          izz="1"/>
+      </inertial>
+      <!--<inertial>-->
+        <!--<mass value="0.015"/>-->
+        <!--<origin xyz="0 0 -${F4_AXLE_HEIGHT-F4_HEIGHT/2+0.0015}" rpy="0 0 0"/>-->
+        <!--[> Full height: (8.2215625e-06, 3.9203124999999996e-06, 6.2612499999999996e-06) <]-->
+        <!--[> Half height: (4.2606249999999995e-06, 3.9203124999999996e-06, 2.3003125e-06) <]-->
+        <!--<inertia ixx="4.261e-6" ixy="0.0" ixz="0.0"-->
+          <!--iyy="3.921e-6" iyz="0.0"-->
+          <!--izz="2.3e-6"/>-->
+      <!--</inertial>-->
       <visual>
         <origin xyz="0 0 0" rpy="${M_PI/2} 0 0"/>
@@ -305,48 +361,62 @@
     <link name="${name}_link">
       <inertial>
-        <mass value="0.02"/>
+        <mass value="0.001"/>
+        <origin xyz="0 0 0.0005" rpy="0 0 0"/>
+        <inertia ixx="1" ixy="0.0" ixz="0.0"
+          iyy="1" iyz="0.0"
+          izz="1"/>
+      </inertial>
+      <!--<inertial>-->
+        <!--<mass value="0.02"/>-->
+        <!--<origin xyz="0 0 0" rpy="0 0 0"/>-->
+        <!--<inertia ixx="1.612e-5" ixy="0.0" ixz="0.0"-->
+          <!--iyy="1.823e-5" iyz="0.0"-->
+          <!--izz="2.732e-6"/>-->
+      <!--</inertial>-->
+      <visual>
         <origin xyz="0 0 0" rpy="0 0 0"/>
-        <inertia ixx="1.612e-5" ixy="0.0" ixz="0.0"
-          iyy="1.823e-5" iyz="0.0"
-          izz="2.732e-6"/>
-      </inertial>
-      <visual>
+        <geometry>
+          <mesh filename="package://crane_plus_description/meshes/finger_fixed.stl" scale="${SCALE_MM} ${SCALE_MM} ${SCALE_MM}"/>
+        </geometry>
+        <material name="${color}"/>
+      </visual>
+      <collision>
         <origin xyz="0 0 0" rpy="0 0 0"/>
         <geometry>
-          <mesh filename="package://crane_plus_description/meshes/finger_fixed.stl" scale="${SCALE_MM} ${SCALE_MM} ${SCALE_MM}"/>
-        </geometry>
-        <material name="${color}"/>
-      </visual>
-      <collision>
+          <mesh filename="package://crane_plus_description/meshes/finger_fixed_collision.stl" scale="${SCALE_MM} ${SCALE_MM} ${SCALE_MM}"/>
+        </geometry>
+      </collision>
+    </link>
+  </xacro:macro>
+  <xacro:macro name="moving_finger" params="parent name color *origin">
+    <joint name="${name}_joint" type="fixed">
+      <xacro:insert_block name="origin"/>
+      <parent link="${parent}"/>
+      <child link="${name}_link"/>
+    </joint>
+    <link name="${name}_link">
+      <inertial>
+        <mass value="0.001"/>
+        <origin xyz="0 0 0.0005" rpy="0 0 0"/>
+        <inertia ixx="1" ixy="0.0" ixz="0.0"
+          iyy="1" iyz="0.0"
+          izz="1"/>
+      </inertial>
+      <!--<inertial>-->
+        <!--<mass value="0.02"/>-->
+        <!--<origin xyz="0 0 0" rpy="0 0 0"/>-->
+        <!--<inertia ixx="2.01e-5" ixy="0.0" ixz="0.0"-->
+          <!--iyy="2.2e-5" iyz="0.0"-->
+          <!--izz="2.936e-6"/>-->
+      <!--</inertial>-->
+      <visual>
         <origin xyz="0 0 0" rpy="0 0 0"/>
         <geometry>
-          <mesh filename="package://crane_plus_description/meshes/finger_fixed_collision.stl" scale="${SCALE_MM} ${SCALE_MM} ${SCALE_MM}"/>
-        </geometry>
-      </collision>
-    </link>
-  </xacro:macro>
-  <xacro:macro name="moving_finger" params="parent name color *origin">
-    <joint name="${name}_joint" type="fixed">
-      <xacro:insert_block name="origin"/>
-      <parent link="${parent}"/>
-      <child link="${name}_link"/>
-    </joint>
-    <link name="${name}_link">
-      <inertial>
-        <mass value="0.02"/>
+          <mesh filename="package://crane_plus_description/meshes/finger_moving.stl" scale="${SCALE_MM} ${SCALE_MM} ${SCALE_MM}"/>
+        </geometry>
+        <material name="${color}"/>
+      </visual>
+      <collision>
         <origin xyz="0 0 0" rpy="0 0 0"/>
-        <inertia ixx="2.01e-5" ixy="0.0" ixz="0.0"
-          iyy="2.2e-5" iyz="0.0"
-          izz="2.936e-6"/>
-      </inertial>
-      <visual>
-        <origin xyz="0 0 0" rpy="0 0 0"/>
-        <geometry>
-          <mesh filename="package://crane_plus_description/meshes/finger_moving.stl" scale="${SCALE_MM} ${SCALE_MM} ${SCALE_MM}"/>
-        </geometry>
-        <material name="${color}"/>
-      </visual>
-      <collision>
-        <origin xyz="0 0 0" rpy="0 0 0"/>
         <geometry>
           <mesh filename="package://crane_plus_description/meshes/finger_moving_collision.stl" scale="${SCALE_MM} ${SCALE_MM} ${SCALE_MM}"/>

File: crane_plus_simulation/urdf/simulated_crane_plus.urdf (robot description, URDF)
Before this commit: robot crane_plus_arm, 20 links, 19 joints
Links:
- link crane_plus_base_bracket_link: mass 0.005 -> 0.001
- link crane_plus_fixed_finger_joiner_link: mass 0.005 -> 0.001
- link crane_plus_fixed_finger_link: mass 0.02 -> 0.001
- link crane_plus_gripper_servo_link: mass 0.0564 -> 0.001
- link crane_plus_lower_arm_bracket_link: mass 0.015 -> 0.001
- link crane_plus_lower_arm_joiner_link: mass 0.005 -> 0.001
- link crane_plus_lower_arm_servo_link: mass 0.0564 -> 0.001
- link crane_plus_mounting_plate_link: mass 0.02 -> 0.001
- link crane_plus_moving_finger_bracket_link: mass 0.01 -> 0.001
- link crane_plus_moving_finger_link: mass 0.02 -> 0.001
- link crane_plus_shoulder_bracket_rev_link: mass 0.01 -> 0.001
- link crane_plus_shoulder_servo_link: mass 0.0564 -> 0.001
- link crane_plus_upper_arm_lower_joiner_link: mass 0.005 -> 0.001
- link crane_plus_upper_arm_servo_link: mass 0.0564 -> 0.001
- link crane_plus_upper_arm_upper_joiner_link: mass 0.005 -> 0.001
- link crane_plus_wrist_bracket_link: mass 0.01 -> 0.001
- link crane_plus_wrist_joiner_link: mass 0.005 -> 0.001
- link crane_plus_wrist_servo_link: mass 0.0564 -> 0.001
