Commit message: Renamed the movable joints to be understandable

File: crane_plus_description/urdf/crane_plus.urdf (robot description, URDF)
Before this commit: robot crane_plus_arm, 20 links, 19 joints
Links:
- removed link crane_plus_lower_arm_bracket_link
- removed link crane_plus_moving_finger_bracket_link
- removed link crane_plus_shoulder_bracket_rev_link
- removed link crane_plus_upper_arm_servo_link
- removed link crane_plus_wrist_bracket_link
- added link gripper_link, mass 0.001; collision box size=0.025 0.0485 0.0375; visual mesh filename=package://crane_plus_description/meshes/f2.stl scale=0.001 0.001 0.001
- added link lower_arm_link, mass 0.001; collision box size=0.028 0.0485 0.065; visual mesh filename=package://crane_plus_description/meshes/f4.stl scale=0.001 0.001 0.001
- added link shoulder_link, mass 0.001; collision box size=0.025 0.0485 0.0375; visual mesh filename=package://crane_plus_description/meshes/f2.stl scale=0.001 0.001 0.001
- added link upper_arm_link, mass 0.001; collision box size=0.05 0.032 0.038; visual mesh filename=package://crane_plus_description/meshes/ax12_box.stl scale=0.001 0.001 0.001
- added link wrist_link, mass 0.001; collision box size=0.025 0.0485 0.0375; visual mesh filename=package://crane_plus_description/meshes/f2.stl scale=0.001 0.001 0.001
Joints:
- removed joint crane_plus_lower_arm_bracket_joint
- removed joint crane_plus_moving_finger_bracket_joint
- removed joint crane_plus_shoulder_bracket_rev_joint
- removed joint crane_plus_upper_arm_servo_joint
- removed joint crane_plus_wrist_bracket_joint
- added joint gripper_joint: type revolute, parent crane_plus_gripper_servo_link, child gripper_link, origin xyz=-0.012 0 0 rpy=-1.570795 0 -1.570795, axis 0 -1 0, limit lower=-2.617 upper=2.617 effort=30 velocity=1.571
- added joint lower_arm_joint: type revolute, parent crane_plus_lower_arm_servo_link, child lower_arm_link, origin xyz=-0.012 0 0 rpy=1.570795 0 1.570795, axis 0 1 0, limit lower=-2.617 upper=2.617 effort=30 velocity=1.571
- added joint shoulder_joint: type revolute, parent crane_plus_shoulder_servo_link, child shoulder_link, origin xyz=-0.0135 0 0.021 rpy=0 0 0, axis 0 0 1, limit lower=-2.617 upper=2.617 effort=30 velocity=1.571
- added joint upper_arm_joint: type revolute, parent shoulder_link, child upper_arm_link, origin xyz=0 0 0.0265 rpy=-1.570795 -1.570795 0, axis 0 0 -1, limit lower=-2.617 upper=2.617 effort=30 velocity=1.571
- added joint wrist_joint: type revolute, parent crane_plus_wrist_servo_link, child wrist_link, origin xyz=-0.012 0 0 rpy=-1.570795 0 -1.570795, axis 0 -1 0, limit lower=-2.617 upper=2.617 effort=30 velocity=1.571
- joint crane_plus_lower_arm_joiner_joint: parent crane_plus_lower_arm_bracket_link -> lower_arm_link
- joint crane_plus_moving_finger_joint: parent crane_plus_moving_finger_bracket_link -> gripper_link
- joint crane_plus_upper_arm_upper_joiner_joint: parent crane_plus_upper_arm_servo_link -> upper_arm_link
- joint crane_plus_wrist_joiner_joint: parent crane_plus_wrist_bracket_link -> wrist_link

File: crane_plus_description/urdf/crane_plus.xacro (robot description, xacro)
@@ -16,4 +16,15 @@
       <child link="crane_plus_base_link"/>
     </joint>
+    <!-- fake gripper_link joint gives us a free servo!
+         this makes us 5DOF and saves you $44.90
+         that's a lot of coin! -->
+    <!--<link name="gripper_link" />-->
+    <!--<joint name="gripper_link_joint" type="revolute">-->
+      <!--<origin xyz="0 0 .112" rpy="0 -1.57 0" />-->
+      <!--<parent link="arm_wrist_flex_link"/>-->
+      <!--<child link="gripper_link" />-->
+      <!--<limit effort="30" velocity="1" lower="-3.14" upper="3.14"/>-->
+      <!--<axis xyz="1 0 0"/>-->
+    <!--</joint>-->
     <!-- Mounting plate -->
     <mounting_plate
@@ -40,5 +51,5 @@
     <bioloid_f2_revolute_base_axis
         parent="crane_plus_shoulder_servo_link"
-        name="crane_plus_shoulder_bracket_rev"
+        name="shoulder"
         color="grey"
         vlimit="${joints_vlimit}"
@@ -49,6 +60,6 @@
     <!--Upper arm servo -->
     <dynamixel_ax12_revolute
-        parent="crane_plus_shoulder_bracket_rev_link"
-        name="crane_plus_upper_arm_servo"
+        parent="shoulder_link"
+        name="upper_arm"
         color="black"
         vlimit="${joints_vlimit}"
@@ -59,5 +70,5 @@
     <!-- Upper arm upper joiner -->
     <bioloid_f3_fixed
-        parent="crane_plus_upper_arm_servo_link"
+        parent="upper_arm_link"
         name="crane_plus_upper_arm_upper_joiner"
         color="grey">
@@ -81,5 +92,5 @@
     <bioloid_f4_revolute
         parent="crane_plus_lower_arm_servo_link"
-        name="crane_plus_lower_arm_bracket"
+        name="lower_arm"
         color="grey"
         vlimit="${joints_vlimit}"
@@ -90,5 +101,5 @@
     <!-- Lower arm joiner -->
     <bioloid_f3_fixed
-        parent="crane_plus_lower_arm_bracket_link"
+        parent="lower_arm_link"
         name="crane_plus_lower_arm_joiner"
         color="grey">
@@ -105,5 +116,5 @@
     <bioloid_f2_revolute
         parent="crane_plus_wrist_servo_link"
-        name="crane_plus_wrist_bracket"
+        name="wrist"
         color="grey"
         vlimit="${joints_vlimit}"
@@ -114,5 +125,5 @@
     <!-- Wrist joiner -->
     <bioloid_f3_fixed
-        parent="crane_plus_wrist_bracket_link"
+        parent="wrist_link"
         name="crane_plus_wrist_joiner"
         color="grey">
@@ -140,8 +151,8 @@
       <origin xyz="0 0 0" rpy="0 0 ${M_PI}"/>
     </fixed_finger>
-    <!-- Wrist bracket -->
+    <!-- Finger bracket -->
     <bioloid_f2_revolute
         parent="crane_plus_gripper_servo_link"
-        name="crane_plus_moving_finger_bracket"
+        name="gripper"
         color="grey"
         vlimit="${joints_vlimit}"
@@ -152,5 +163,5 @@
     <!-- Movin finger -->
     <moving_finger
-        parent="crane_plus_moving_finger_bracket_link"
+        parent="gripper_link"
         name="crane_plus_moving_finger"
         color="black">

File: crane_plus_description/urdf/crane_plus_hardware.xacro (robot description, xacro)
@@ -160,5 +160,5 @@
     <joint name="${name}_joint" type="revolute">
       <xacro:insert_block name="origin"/>
-      <axis xyz="0 0 1"/>
+      <axis xyz="0 0 -1"/>
       <limit effort="30" velocity="${vlimit}" lower="${llimit}" upper="${ulimit}"/>
       <parent link="${parent}"/>
@@ -238,5 +238,5 @@
     <joint name="${name}_joint" type="revolute">
       <xacro:insert_block name="origin"/>
-      <axis xyz="0 1 0"/>
+      <axis xyz="0 -1 0"/>
       <limit effort="30" velocity="${vlimit}" lower="${llimit}" upper="${ulimit}"/>
       <parent link="${parent}"/>

Commit message: Fixed MoveIt config and set correct joint limits

File: crane_plus_description/urdf/crane_plus.urdf (robot description, URDF)
Before this commit: robot crane_plus_arm, 20 links, 19 joints
Joints:
- joint gripper_joint: limit lower=-2.617 upper=2.617 effort=30 velocity=1.571 -> lower=-3.14159 upper=3.14159 effort=30 velocity=1.571
- joint lower_arm_joint: limit lower=-2.617 upper=2.617 effort=30 velocity=1.571 -> lower=-3.14159 upper=3.14159 effort=30 velocity=1.571
- joint shoulder_joint: limit lower=-2.617 upper=2.617 effort=30 velocity=1.571 -> lower=-3.14159 upper=3.14159 effort=30 velocity=1.571
- joint upper_arm_joint: limit lower=-2.617 upper=2.617 effort=30 velocity=1.571 -> lower=-3.14159 upper=3.14159 effort=30 velocity=1.571
- joint wrist_joint: limit lower=-2.617 upper=2.617 effort=30 velocity=1.571 -> lower=-3.14159 upper=3.14159 effort=30 velocity=1.571

File: crane_plus_description/urdf/crane_plus.xacro (robot description, xacro)
@@ -3,5 +3,5 @@
   <xacro:include filename="$(find crane_plus_description)/urdf/crane_plus_hardware.xacro"/>
   <material name="grey">
-    <color rgba="0.6 0.6 0.6 1.0"/>
+    <color rgba="0.75 0.75 0.75 1.0"/>
   </material>
   <material name="black">
@@ -16,12 +16,10 @@
       <child link="crane_plus_base_link"/>
     </joint>
-    <!-- fake gripper_link joint gives us a free servo!
-         this makes us 5DOF and saves you $44.90
-         that's a lot of coin! -->
-    <!--<link name="gripper_link" />-->
-    <!--<joint name="gripper_link_joint" type="revolute">-->
-      <!--<origin xyz="0 0 .112" rpy="0 -1.57 0" />-->
-      <!--<parent link="arm_wrist_flex_link"/>-->
-      <!--<child link="gripper_link" />-->
+    <!-- fake gripper_link joint gives us a free servo, making the arm 5DOF -->
+    <!--<link name="virtual_gripper_link" />-->
+    <!--<joint name="virtual_gripper_joint" type="revolute">-->
+      <!--<origin xyz="-0.015 0 0.1" rpy="0 -1.57 0" />-->
+      <!--<parent link="crane_plus_wrist_joiner_link"/>-->
+      <!--<child link="virtual_gripper_link" />-->
       <!--<limit effort="30" velocity="1" lower="-3.14" upper="3.14"/>-->
       <!--<axis xyz="1 0 0"/>-->
@@ -64,6 +62,6 @@
         color="black"
         vlimit="${joints_vlimit}"
-        llimit="${pan_llimit}"
-        ulimit="${pan_ulimit}">
+        llimit="-1.7"
+        ulimit="1.7">
         <origin xyz="0 0 ${F2_AXLE_HEIGHT}" rpy="-${M_PI/2} -${M_PI/2} 0"/>
     </dynamixel_ax12_revolute>
@@ -95,6 +93,6 @@
         color="grey"
         vlimit="${joints_vlimit}"
-        llimit="${pan_llimit}"
-        ulimit="${pan_ulimit}">
+        llimit="-2.3"
+        ulimit="2.3">
         <origin xyz="-${AX12_ORIGIN_TO_AXLE} 0 0" rpy="${M_PI/2} 0 ${M_PI/2}"/>
     </bioloid_f4_revolute>
@@ -119,6 +117,6 @@
         color="grey"
         vlimit="${joints_vlimit}"
-        llimit="${pan_llimit}"
-        ulimit="${pan_ulimit}">
+        llimit="-1.7"
+        ulimit="1.7">
         <origin xyz="-${AX12_ORIGIN_TO_AXLE} 0 0" rpy="-${M_PI/2} 0 -${M_PI/2}"/>
     </bioloid_f2_revolute>
@@ -151,5 +149,5 @@
       <origin xyz="0 0 0" rpy="0 0 ${M_PI}"/>
     </fixed_finger>
-    <!-- Finger bracket -->
+    <!-- Finger bracket (actual gripper joint) -->
     <bioloid_f2_revolute
         parent="crane_plus_gripper_servo_link"
@@ -157,6 +155,6 @@
         color="grey"
         vlimit="${joints_vlimit}"
-        llimit="${pan_llimit}"
-        ulimit="${pan_ulimit}">
+        llimit="0.6"
+        ulimit="0.65">
         <origin xyz="-${AX12_ORIGIN_TO_AXLE} 0 0" rpy="-${M_PI/2} 0 -${M_PI/2}"/>
     </bioloid_f2_revolute>
