Commit message: Working on joint names reorganisation and simulated gripper

File: crane_plus_description/urdf/crane_plus.urdf (robot description, URDF)
Before this commit: robot crane_plus_arm, 20 links, 19 joints
Links:
- removed link crane_plus_base_bracket_link
- removed link crane_plus_fixed_finger_joiner_link
- removed link crane_plus_fixed_finger_link
- removed link crane_plus_gripper_servo_link
- removed link crane_plus_lower_arm_joiner_link
- removed link crane_plus_lower_arm_servo_link
- removed link crane_plus_mounting_plate_link
- removed link crane_plus_shoulder_servo_link
- removed link crane_plus_upper_arm_lower_joiner_link
- removed link crane_plus_upper_arm_upper_joiner_link
- removed link crane_plus_wrist_joiner_link
- removed link crane_plus_wrist_servo_link
- removed link gripper_link
- removed link lower_arm_link
- removed link shoulder_link
- removed link upper_arm_link
- removed link wrist_link
- added link crane_plus_elbow_link, mass 0.001; collision box size=0.028 0.0485 0.065; visual mesh filename=package://crane_plus_description/meshes/f4.stl scale=0.001 0.001 0.001
- added link crane_plus_fixed_finger_tip_link
- added link crane_plus_gripper_centre
- added link crane_plus_internal_base_bracket_link, mass 0.001; collision box size=0.022 0.032 0.008; visual mesh filename=package://crane_plus_description/meshes/f53.stl scale=0.01 0.01 0.01
- added link crane_plus_internal_fixed_finger_joiner_link, mass 0.001; collision box size=0.025 0.038 0.009; visual mesh filename=package://crane_plus_description/meshes/f3.stl scale=0.001 0.001 0.001
- added link crane_plus_internal_fixed_finger_link, mass 0.001; collision mesh filename=package://crane_plus_description/meshes/finger_fixed_collis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 scale=0.001 0.001 0.001; visual mesh filename=package://crane_plus_description/meshes/finger_fixed.stl scale=0.001 0.001 0.001
- added link crane_plus_internal_gripper_servo_link, mass 0.001; collision box size=0.05 0.032 0.038; visual mesh filename=package://crane_plus_description/meshes/ax12_box.stl scale=0.001 0.001 0.001
- added link crane_plus_internal_lower_arm_joiner_link, mass 0.001; collision box size=0.025 0.038 0.009; visual mesh filename=package://crane_plus_description/meshes/f3.stl scale=0.001 0.001 0.001
- added link crane_plus_internal_lower_arm_servo_link, mass 0.001; collision box size=0.05 0.032 0.038; visual mesh filename=package://crane_plus_description/meshes/ax12_box.stl scale=0.001 0.001 0.001
- added link crane_plus_internal_mounting_plate_link, mass 0.001; collision box size=0.05 0.05 0.001; visual mesh filename=package://crane_plus_description/meshes/mount.stl scale=1 1 1
- added link crane_plus_internal_moving_finger_plate_link, mass 0.001; collision mesh filename=package://crane_plus_description/meshes/finger_moving_colli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 scale=0.001 0.001 0.001; visual mesh filename=package://crane_plus_description/meshes/finger_moving.stl scale=0.001 0.001 0.001
- added link crane_plus_internal_shoulder_servo_link, mass 0.001; collision box size=0.05 0.032 0.038; visual mesh filename=package://crane_plus_description/meshes/ax12_box.stl scale=0.001 0.001 0.001
- added link crane_plus_internal_upper_arm_lower_joiner_link, mass 0.001; collision box size=0.025 0.038 0.009; visual mesh filename=package://crane_plus_description/meshes/f3.stl scale=0.001 0.001 0.001
- added link crane_plus_internal_upper_arm_upper_joiner_link, mass 0.001; collision box size=0.025 0.038 0.009; visual mesh filename=package://crane_plus_description/meshes/f3.stl scale=0.001 0.001 0.001
- added link crane_plus_internal_wrist_joiner_link, mass 0.001; collision box size=0.025 0.038 0.009; visual mesh filename=package://crane_plus_description/meshes/f3.stl scale=0.001 0.001 0.001
- added link crane_plus_internal_wrist_servo_link, mass 0.001; collision box size=0.05 0.032 0.038; visual mesh filename=package://crane_plus_description/meshes/ax12_box.stl scale=0.001 0.001 0.001
- added link crane_plus_moving_finger_tip_link
- added link crane_plus_shoulder_flex_link, mass 0.001; collision box size=0.05 0.032 0.038; visual mesh filename=package://crane_plus_description/meshes/ax12_box.stl scale=0.001 0.001 0.001
- added link crane_plus_shoulder_revolute_link, mass 0.001; collision box size=0.025 0.0485 0.0375; visual mesh filename=package://crane_plus_description/meshes/f2.stl scale=0.001 0.001 0.001
- added link crane_plus_wrist_link, mass 0.001; collision box size=0.025 0.0485 0.0375; visual mesh filename=package://crane_plus_description/meshes/f2.stl scale=0.001 0.001 0.001
- link crane_plus_moving_finger_link: geometry collision box size=0.025 0.0485 0.0375; visual mesh filename=package://crane_plus_description/meshes/f2.stl scale=0.001 0.001 0.001
Joints:
- removed joint crane_plus_base_bracket_joint
- removed joint crane_plus_fixed_finger_joiner_joint
- removed joint crane_plus_fixed_finger_joint
- removed joint crane_plus_gripper_servo_joint
- removed joint crane_plus_lower_arm_joiner_joint
- removed joint crane_plus_lower_arm_servo_joint
- removed joint crane_plus_mounting_plate_joint
- removed joint crane_plus_shoulder_servo_joint
- removed joint crane_plus_upper_arm_lower_joiner_joint
- removed joint crane_plus_upper_arm_upper_joiner_joint
- removed joint crane_plus_wrist_joiner_joint
- removed joint crane_plus_wrist_servo_joint
- removed joint gripper_joint
- removed joint lower_arm_joint
- removed joint shoulder_joint
- removed joint upper_arm_joint
- removed joint wrist_joint
- added joint crane_plus_elbow_joint: type revolute, parent crane_plus_internal_lower_arm_servo_link, child crane_plus_elbow_link, origin xyz=-0.012 0 0 rpy=1.570795 0 1.570795, axis 0 1 0, limit lower=-2.3 upper=2.3 effort=30 velocity=1.571
- added joint crane_plus_fixed_finger_tip: type fixed, parent crane_plus_internal_fixed_finger_link, child crane_plus_fixed_finger_tip_link, origin xyz=0.0745 0 -0.0106 rpy=1.570795 0 1.570795
- added joint crane_plus_gripper_joint: type fixed, parent crane_plus_internal_gripper_servo_link, child crane_plus_gripper_centre, origin xyz=0 -0.0537 0 rpy=1.570795 -1.570795 0
- added joint crane_plus_internal_base_bracket_joint: type fixed, parent crane_plus_internal_mounting_plate_link, child crane_plus_internal_base_bracket_link, origin xyz=0 0 0.001 rpy=0 0 0
- added joint crane_plus_internal_fixed_finger_joiner_joint: type fixed, parent crane_plus_internal_gripper_servo_link, child crane_plus_internal_fixed_finger_joiner_link, origin xyz=0.0295 0 0 rpy=-1.570795 0 1.570795
- added joint crane_plus_internal_fixed_finger_joint: type fixed, parent crane_plus_internal_fixed_finger_joiner_link, child crane_plus_internal_fixed_finger_link, origin xyz=0 0 0 rpy=0 0 3.14159
- added joint crane_plus_internal_gripper_servo_joint: type fixed, parent crane_plus_internal_wrist_joiner_link, child crane_plus_internal_gripper_servo_link, origin xyz=0.0028 0 0.019 rpy=1.570795 3.14159 0
- added joint crane_plus_internal_lower_arm_joiner_joint: type fixed, parent crane_plus_elbow_link, child crane_plus_internal_lower_arm_joiner_link, origin xyz=0 0 -0.0525 rpy=0 3.14159 0
- added joint crane_plus_internal_lower_arm_servo_joint: type fixed, parent crane_plus_internal_upper_arm_lower_joiner_link, child crane_plus_internal_lower_arm_servo_link, origin xyz=0 0 0.0295 rpy=0 1.570795 1.570795
- added joint crane_plus_internal_mounting_plate_joint: type fixed, parent crane_plus_base_link, child crane_plus_internal_mounting_plate_link, origin xyz=0 0 0 rpy=0 0 0
- added joint crane_plus_internal_moving_finger_plate_joint: type fixed, parent crane_plus_moving_finger_link, child crane_plus_internal_moving_finger_plate_link, origin xyz=0 0 -0.0265 rpy=3.14159 0 0
- added joint crane_plus_internal_shoulder_servo_joint: type fixed, parent crane_plus_internal_base_bracket_link, child crane_plus_internal_shoulder_servo_link, origin xyz=-0.0028 0 0.023 rpy=0 0 0
- added joint crane_plus_internal_upper_arm_lower_joiner_joint: type fixed, parent crane_plus_internal_upper_arm_upper_joiner_link, child crane_plus_internal_upper_arm_lower_joiner_link, origin xyz=0 0 0 rpy=3.14159 0 0
- added joint crane_plus_internal_upper_arm_upper_joiner_joint: type fixed, parent crane_plus_shoulder_flex_link, child crane_plus_internal_upper_arm_upper_joiner_link, origin xyz=0.0415 0 0 rpy=-1.570795 0 1.570795
- added joint crane_plus_internal_wrist_joiner_joint: type fixed, parent crane_plus_wrist_link, child crane_plus_internal_wrist_joiner_link, origin xyz=0 0 -0.0265 rpy=0 3.14159 1.570795
- added joint crane_plus_internal_wrist_servo_joint: type fixed, parent crane_plus_internal_lower_arm_joiner_link, child crane_plus_internal_wrist_servo_link, origin xyz=0 0 0.0295 rpy=0 1.570795 1.570795
- added joint crane_plus_moving_finger_tip: type fixed, parent crane_plus_internal_moving_finger_plate_link, child crane_plus_moving_finger_tip_link, origin xyz=0.0923 0 -0.0194 rpy=1.570795 0 1.570795
- added joint crane_plus_shoulder_flex_joint: type revolute, parent crane_plus_shoulder_revolute_link, child crane_plus_shoulder_flex_link, origin xyz=0 0 0.0265 rpy=-1.570795 -1.570795 0, axis 0 0 -1, limit lower=-1.7 upper=1.7 effort=30 velocity=1.571
- added joint crane_plus_shoulder_revolute_joint: type revolute, parent crane_plus_internal_shoulder_servo_link, child crane_plus_shoulder_revolute_link, origin xyz=-0.0135 0 0.021 rpy=0 0 0, axis 0 0 1, limit lower=-2.617 upper=2.617 effort=30 velocity=1.571
- added joint crane_plus_wrist_joint: type revolute, parent crane_plus_internal_wrist_servo_link, child crane_plus_wrist_link, origin xyz=-0.012 0 0 rpy=-1.570795 0 -1.570795, axis 0 -1 0, limit lower=-1.7 upper=1.7 effort=30 velocity=1.571
- joint crane_plus_moving_finger_joint: axis (none) -> 0 -1 0; limit (none) -> lower=-0.6 upper=0.65 effort=30 velocity=1.571; origin xyz=0 0 -0.0265 rpy=3.14159 0 0 -> xyz=-0.012 0 0 rpy=-1.570795 0 -1.570795; parent gripper_link -> crane_plus_internal_gripper_servo_link; type fixed -> revolute

File: crane_plus_description/urdf/crane_plus.xacro (robot description, xacro)
@@ -16,17 +16,10 @@
       <child link="crane_plus_base_link"/>
     </joint>
-    <!-- fake gripper_link joint gives us a free servo, making the arm 5DOF -->
-    <!--<link name="virtual_gripper_link" />-->
-    <!--<joint name="virtual_gripper_joint" type="revolute">-->
-      <!--<origin xyz="-0.015 0 0.1" rpy="0 -1.57 0" />-->
-      <!--<parent link="crane_plus_wrist_joiner_link"/>-->
-      <!--<child link="virtual_gripper_link" />-->
-      <!--<limit effort="30" velocity="1" lower="-3.14" upper="3.14"/>-->
-      <!--<axis xyz="1 0 0"/>-->
-    <!--</joint>-->
+    <!-- TODO: When rviz supports multiple materials per link, combine the
+         meshes to simplify the link structure. -->
     <!-- Mounting plate -->
     <mounting_plate
         parent="crane_plus_base_link"
-        name="crane_plus_mounting_plate"
+        name="crane_plus_internal_mounting_plate"
         color="black">
       <origin xyz="0 0 0" rpy="0 0 0"/>
@@ -34,6 +27,6 @@
     <!-- Base bracket -->
     <bioloid_f53_fixed
-        parent="crane_plus_mounting_plate_link"
-        name="crane_plus_base_bracket"
+        parent="crane_plus_internal_mounting_plate_link"
+        name="crane_plus_internal_base_bracket"
         color="grey">
       <origin xyz="0 0 ${MOUNT_HEIGHT}" rpy="0 0 0"/>
@@ -41,6 +34,6 @@
     <!-- Shoulder servo -->
     <dynamixel_ax12_fixed
-        parent="crane_plus_base_bracket_link"
-        name="crane_plus_shoulder_servo"
+        parent="crane_plus_internal_base_bracket_link"
+        name="crane_plus_internal_shoulder_servo"
         color="black">
         <origin xyz="-${AX12_SIDE_SCREW_OFFSET} 0 ${AX12_BODY_MAIN_HEIGHT/2 + F53_HEIGHT}" rpy="0 0 0"/>
@@ -48,6 +41,6 @@
     <!-- Shoulder bracket -->
     <bioloid_f2_revolute_base_axis
-        parent="crane_plus_shoulder_servo_link"
-        name="shoulder"
+        parent="crane_plus_internal_shoulder_servo_link"
+        name="crane_plus_shoulder_revolute"
         color="grey"
         vlimit="${joints_vlimit}"
@@ -58,6 +51,6 @@
     <!--Upper arm servo -->
     <dynamixel_ax12_revolute
-        parent="shoulder_link"
-        name="upper_arm"
+        parent="crane_plus_shoulder_revolute_link"
+        name="crane_plus_shoulder_flex"
         color="black"
         vlimit="${joints_vlimit}"
@@ -68,6 +61,6 @@
     <!-- Upper arm upper joiner -->
     <bioloid_f3_fixed
-        parent="upper_arm_link"
-        name="crane_plus_upper_arm_upper_joiner"
+        parent="crane_plus_shoulder_flex_link"
+        name="crane_plus_internal_upper_arm_upper_joiner"
         color="grey">
         <origin xyz="${AX12_ORIGIN_TO_AXLE+AX12_ORIGIN_TO_END_SCREW+F3_SCREW_HEIGHT} 0 0" rpy="-${M_PI/2} 0 ${M_PI/2}"/>
@@ -75,6 +68,6 @@
     <!-- Upper arm lower joiner -->
     <bioloid_f3_fixed
-        parent="crane_plus_upper_arm_upper_joiner_link"
-        name="crane_plus_upper_arm_lower_joiner"
+        parent="crane_plus_internal_upper_arm_upper_joiner_link"
+        name="crane_plus_internal_upper_arm_lower_joiner"
         color="grey">
         <origin xyz="0 0 0" rpy="${M_PI} 0 0"/>
@@ -82,6 +75,6 @@
     <!-- Lower arm servo -->
     <dynamixel_ax12_fixed
-        parent="crane_plus_upper_arm_lower_joiner_link"
-        name="crane_plus_lower_arm_servo"
+        parent="crane_plus_internal_upper_arm_lower_joiner_link"
+        name="crane_plus_internal_lower_arm_servo"
         color="black">
       <origin xyz="0 0 ${F3_SCREW_HEIGHT+AX12_ORIGIN_TO_END_SCREW}" rpy="0 ${M_PI/2} ${M_PI/2}"/>
@@ -89,6 +82,6 @@
     <!-- Lower arm bracket -->
     <bioloid_f4_revolute
-        parent="crane_plus_lower_arm_servo_link"
-        name="lower_arm"
+        parent="crane_plus_internal_lower_arm_servo_link"
+        name="crane_plus_elbow"
         color="grey"
         vlimit="${joints_vlimit}"
@@ -99,6 +92,6 @@
     <!-- Lower arm joiner -->
     <bioloid_f3_fixed
-        parent="lower_arm_link"
-        name="crane_plus_lower_arm_joiner"
+        parent="crane_plus_elbow_link"
+        name="crane_plus_internal_lower_arm_joiner"
         color="grey">
         <origin xyz="0 0 -${F4_AXLE_HEIGHT}" rpy="0 ${M_PI} 0"/>
@@ -106,6 +99,6 @@
     <!-- Wrist servo -->
     <dynamixel_ax12_fixed
-        parent="crane_plus_lower_arm_joiner_link"
-        name="crane_plus_wrist_servo"
+        parent="crane_plus_internal_lower_arm_joiner_link"
+        name="crane_plus_internal_wrist_servo"
         color="black">
       <origin xyz="0 0 ${F3_SCREW_HEIGHT+AX12_ORIGIN_TO_END_SCREW}" rpy="0 ${M_PI/2} ${M_PI/2}"/>
@@ -113,6 +106,6 @@
     <!-- Wrist bracket -->
     <bioloid_f2_revolute
-        parent="crane_plus_wrist_servo_link"
-        name="wrist"
+        parent="crane_plus_internal_wrist_servo_link"
+        name="crane_plus_wrist"
         color="grey"
         vlimit="${joints_vlimit}"
@@ -123,6 +116,6 @@
     <!-- Wrist joiner -->
     <bioloid_f3_fixed
-        parent="wrist_link"
-        name="crane_plus_wrist_joiner"
+        parent="crane_plus_wrist_link"
+        name="crane_plus_internal_wrist_joiner"
         color="grey">
         <origin xyz="0 0 -${F2_AXLE_HEIGHT}" rpy="0 ${M_PI} ${M_PI/2}"/>
@@ -130,6 +123,6 @@
     <!-- Gripper servo -->
     <dynamixel_ax12_fixed
-        parent="crane_plus_wrist_joiner_link"
-        name="crane_plus_gripper_servo"
+        parent="crane_plus_internal_wrist_joiner_link"
+        name="crane_plus_internal_gripper_servo"
         color="black">
         <origin xyz="${AX12_SIDE_SCREW_OFFSET} 0 ${F3_SCREW_HEIGHT+AX12_ORIGIN_TO_SIDE_SCREW}" rpy="${M_PI/2} ${M_PI} 0"/>
@@ -137,6 +130,6 @@
     <!-- Fixed finger joiner -->
     <bioloid_f3_fixed
-        parent="crane_plus_gripper_servo_link"
-        name="crane_plus_fixed_finger_joiner"
+        parent="crane_plus_internal_gripper_servo_link"
+        name="crane_plus_internal_fixed_finger_joiner"
         color="grey">
         <origin xyz="${AX12_ORIGIN_TO_END_SCREW+F3_SCREW_HEIGHT} 0 0" rpy="-${M_PI/2} 0 ${M_PI/2}"/>
@@ -144,13 +137,20 @@
     <!-- Fixed finger -->
     <fixed_finger
-        parent="crane_plus_fixed_finger_joiner_link"
-        name="crane_plus_fixed_finger"
+        parent="crane_plus_internal_fixed_finger_joiner_link"
+        name="crane_plus_internal_fixed_finger"
         color="black">
       <origin xyz="0 0 0" rpy="0 0 ${M_PI}"/>
     </fixed_finger>
-    <!-- Finger bracket (actual gripper joint) -->
+    <!-- Tip of the fixed finger (useful in all sorts of ways) -->
+    <joint name="crane_plus_fixed_finger_tip" type="fixed">
+      <origin xyz="0.0745 0 -0.0106" rpy="${M_PI/2} 0 ${M_PI/2}"/>
+      <parent link="crane_plus_internal_fixed_finger_link"/>
+      <child link="crane_plus_fixed_finger_tip_link"/>
+    </joint>
+    <link name="crane_plus_fixed_finger_tip_link"/>
+    <!-- Moving finger bracket (actual gripper joint) -->
     <bioloid_f2_revolute
-        parent="crane_plus_gripper_servo_link"
-        name="gripper"
+        parent="crane_plus_internal_gripper_servo_link"
+        name="crane_plus_moving_finger"
         color="grey"
         vlimit="${joints_vlimit}"
@@ -161,9 +161,23 @@
     <!-- Moving finger -->
     <moving_finger
-        parent="gripper_link"
-        name="crane_plus_moving_finger"
+        parent="crane_plus_moving_finger_link"
+        name="crane_plus_internal_moving_finger_plate"
         color="black">
       <origin xyz="0 0 -${F2_AXLE_HEIGHT}" rpy="${M_PI} 0 0"/>
     </moving_finger>
+    <!-- Tip of the moving finger (useful in all sorts of ways) -->
+    <joint name="crane_plus_moving_finger_tip" type="fixed">
+      <origin xyz="0.0923 0 -0.0194" rpy="${M_PI/2} 0 ${M_PI/2}"/>
+      <parent link="crane_plus_internal_moving_finger_plate_link"/>
+      <child link="crane_plus_moving_finger_tip_link"/>
+    </joint>
+    <link name="crane_plus_moving_finger_tip_link"/>
+    <!-- A virtual link to make it easy to find the centre of the gripper -->
+    <link name="crane_plus_gripper_centre"/>
+    <joint name="crane_plus_gripper_joint" type="fixed">
+      <origin xyz="0 -0.0537 0" rpy="${M_PI/2} -${M_PI/2} 0"/>
+      <parent link="crane_plus_internal_gripper_servo_link"/>
+      <child link="crane_plus_gripper_centre" />
+    </joint>
   </xacro:macro>
 </robot>

File: crane_plus_simulation/urdf/simulated_crane_plus.urdf.xacro (robot description, xacro)
@@ -22,33 +22,33 @@
   </crane_plus>
   <!-- Add the transmissions necessary to move the simulated robot's joints -->
-  <!-- Shoulder servo -->
-  <transmission name="shoulder">
+  <!-- Shoulder revolute servo -->
+  <transmission name="shoulder_revolute">
     <type>transmission_interface/SimpleTransmission</type>
-    <joint name="shoulder_joint">
+    <joint name="crane_plus_shoulder_revolute_joint">
       <hardwareInterface>PositionJointInterface</hardwareInterface>
     </joint>
-    <actuator name="shoulder_servo">
+    <actuator name="shoulder_revolute_servo">
       <hardwareInterface>PositionJointInterface</hardwareInterface>
       <mechanicalReduction>1</mechanicalReduction>
     </actuator>
   </transmission>
-  <!-- Upper arm servo -->
-  <transmission name="upper_arm">
+  <!-- Shoulder flex servo -->
+  <transmission name="shoulder_flex">
     <type>transmission_interface/SimpleTransmission</type>
-    <joint name="upper_arm_joint">
+    <joint name="crane_plus_shoulder_flex_joint">
       <hardwareInterface>PositionJointInterface</hardwareInterface>
     </joint>
-    <actuator name="upper_arm_servo">
+    <actuator name="shoulder_flex_servo">
       <hardwareInterface>PositionJointInterface</hardwareInterface>
       <mechanicalReduction>1</mechanicalReduction>
     </actuator>
   </transmission>
-  <!-- Lower arm servo -->
-  <transmission name="lower_arm">
+  <!-- Elbow servo -->
+  <transmission name="elbow">
     <type>transmission_interface/SimpleTransmission</type>
-    <joint name="lower_arm_joint">
+    <joint name="crane_plus_elbow_joint">
       <hardwareInterface>PositionJointInterface</hardwareInterface>
     </joint>
-    <actuator name="lower_arm_servo">
+    <actuator name="elbow_servo">
       <hardwareInterface>PositionJointInterface</hardwareInterface>
       <mechanicalReduction>1</mechanicalReduction>
@@ -58,5 +58,5 @@
   <transmission name="wrist">
     <type>transmission_interface/SimpleTransmission</type>
-    <joint name="wrist_joint">
+    <joint name="crane_plus_wrist_joint">
       <hardwareInterface>PositionJointInterface</hardwareInterface>
     </joint>
@@ -66,11 +66,11 @@
     </actuator>
   </transmission>
-  <!-- Gripper servo -->
-  <transmission name="gripper">
+  <!-- Finger servo -->
+  <transmission name="finger">
     <type>transmission_interface/SimpleTransmission</type>
-    <joint name="gripper_joint">
+    <joint name="crane_plus_moving_finger_joint">
       <hardwareInterface>PositionJointInterface</hardwareInterface>
     </joint>
-    <actuator name="gripper_servo">
+    <actuator name="finger_servo">
       <hardwareInterface>PositionJointInterface</hardwareInterface>
       <mechanicalReduction>1</mechanicalReduction>
@@ -81,9 +81,9 @@
     <plugin name="joint_state_publisher" filename="libgazebo_ros_joint_state_publisher.so">
       <jointName>
-        shoulder_joint,
-        upper_arm_joint,
-        lower_arm_joint,
-        wrist_joint,
-        gripper_joint
+        crane_plus_shoulder_revolute_joint,
+        crane_plus_shoulder_flex_joint,
+        crane_plus_elbow_joint,
+        crane_plus_wrist_joint,
+        crane_plus_moving_finger_joint
       </jointName>
     </plugin>
