Commit message: Generated ikfast plugin for moveit

File: crane_plus_description/urdf/crane_plus.urdf (robot description, URDF)
Before this commit: robot crane_plus_arm, 23 links, 22 joints
Links:
- removed link crane_plus_base_link
- removed link crane_plus_gripper_centre
- removed link world
- added link base_link
- added link crane_plus_gripper_link
- added link crane_plus_mounting_link
Joints:
- removed joint crane_plus_base_joint
- added joint crane_plus_mounting_joint: type fixed, parent base_link, child crane_plus_mounting_link, origin xyz=0 0 0
- joint crane_plus_gripper_joint: axis (none) -> 1 0 0; child crane_plus_gripper_centre -> crane_plus_gripper_link; limit (none) -> lower=-3.14159 upper=3.14159 effort=30 velocity=1; origin xyz=0 -0.0537 0 rpy=1.570795 -1.570795 0 -> xyz=0 0 0.0537 rpy=0 0 -1.570795; parent crane_plus_internal_gripper_servo_link -> crane_plus_internal_wrist_joiner_link; type fixed -> revolute
- joint crane_plus_internal_mounting_plate_joint: parent crane_plus_base_link -> crane_plus_mounting_link

File: crane_plus_description/urdf/crane_plus.urdf.xacro (robot description, xacro)
@@ -1,5 +1,5 @@
 <?xml version="1.0"?>
 <robot
-    name="crane_plus_arm"
+    name="crane_plus"
     xmlns:xacro="http://ros.org/wiki/xacro"
     xmlns:sensor="http://playerstage.sourceforge.net/gazebo/xmlschema/#sensor"
@@ -9,10 +9,10 @@
   <xacro:include filename="$(find crane_plus_description)/urdf/crane_plus.xacro"/>
   <!-- Link to provide the location reference for the arm -->
-  <link name="world"/>
+  <link name="base_link"/>
   <!-- Use the crane_plus macro to configure a Crane+ arm with desired joint
        velocities limit and lower/upper limits for the first joint. This
        allows accessing different operational areas, e.g. left-handed vs.
        right-handed robots. -->
-  <crane_plus parent="world"
+  <crane_plus parent="base_link"
               servo_color="black" bracket_color="grey" gripper_color="black"
               joints_vlimit="1.571"

File: crane_plus_description/urdf/crane_plus.xacro (robot description, xacro)
@@ -10,9 +10,9 @@
   <xacro:macro name="crane_plus" params="parent servo_color bracket_color
                gripper_color *origin joints_vlimit pan_llimit pan_ulimit">
-    <link name="crane_plus_base_link"/>
-    <joint name="crane_plus_base_joint" type="fixed">
+    <link name="crane_plus_mounting_link"/>
+    <joint name="crane_plus_mounting_joint" type="fixed">
       <xacro:insert_block name="origin"/>
       <parent link="${parent}"/>
-      <child link="crane_plus_base_link"/>
+      <child link="crane_plus_mounting_link"/>
     </joint>
     <!-- TODO: When rviz supports multiple materials per link, combine the
@@ -20,5 +20,5 @@
     <!-- Mounting plate -->
     <mounting_plate
-        parent="crane_plus_base_link"
+        parent="crane_plus_mounting_link"
         name="crane_plus_internal_mounting_plate"
         color="black">
@@ -173,10 +173,13 @@
     </joint>
     <link name="crane_plus_moving_finger_tip_link"/>
-    <!-- A virtual link to make it easy to find the centre of the gripper -->
-    <link name="crane_plus_gripper_centre"/>
-    <joint name="crane_plus_gripper_joint" type="fixed">
-      <origin xyz="0 -0.0537 0" rpy="${M_PI/2} -${M_PI/2} 0"/>
-      <parent link="crane_plus_internal_gripper_servo_link"/>
-      <child link="crane_plus_gripper_centre" />
+    <!-- A virtual link for the gripper to hang off, increasing the degrees of
+         freedom by one and making it easier for MoveIt! to plan. -->
+    <link name="crane_plus_gripper_link"/>
+    <joint name="crane_plus_gripper_joint" type="revolute">
+      <origin xyz="0 0 0.0537" rpy="0 0 -${M_PI/2}"/>
+      <axis xyz="1 0 0"/>
+      <parent link="crane_plus_internal_wrist_joiner_link"/>
+      <child link="crane_plus_gripper_link" />
+      <limit effort="30" velocity="1" lower="-${M_PI}" upper="${M_PI}"/>
     </joint>
   </xacro:macro>

File: crane_plus_simulation/urdf/simulated_crane_plus.urdf.xacro (robot description, xacro)
@@ -1,5 +1,5 @@
 <?xml version="1.0"?>
 <robot
-    name="crane_plus_arm"
+    name="crane_plus"
     xmlns:xacro="http://ros.org/wiki/xacro"
     xmlns:sensor="http://playerstage.sourceforge.net/gazebo/xmlschema/#sensor"
