Commit message: Move fake gripper link out ~1.5 cm

File: crane_plus_description/urdf/crane_plus.xacro (robot description, xacro)
@@ -177,5 +177,5 @@
     <link name="crane_plus_gripper_link"/>
     <joint name="crane_plus_gripper_joint" type="revolute">
-      <origin xyz="0 0 0.0537" rpy="0 0 -${M_PI/2}"/>
+      <origin xyz="0 0 0.07" rpy="0 0 -${M_PI/2}"/>
       <axis xyz="1 0 0"/>
       <parent link="crane_plus_internal_wrist_joiner_link"/>
