Commit message: Working on simulation package

File: crane_plus_description/urdf/crane_plus.urdf.xacro (robot description, xacro)
@@ -1,24 +1,26 @@
 <?xml version="1.0"?>
-<robot name="crane_plus_arm" xmlns:xacro="http://ros.org/wiki/xacro"
+<robot
+    name="crane_plus_arm"
+    xmlns:xacro="http://ros.org/wiki/xacro"
     xmlns:sensor="http://playerstage.sourceforge.net/gazebo/xmlschema/#sensor"
     xmlns:controller="http://playerstage.sourceforge.net/gazebo/xmlschema/#controller"
     xmlns:interface="http://playerstage.sourceforge.net/gazebo/xmlschema/#interface">
-    <!-- Included URDF Files -->
-    <xacro:include filename="$(find crane_plus_description)/urdf/crane_plus.xacro"/>
-    <!-- Link to provide the location reference for the arm -->
-    <link name="base_link"/>
-    <!-- Use the crane_plus macro to configure a Crane+ arm with desired joint
-         velocities limit and lower/upper limits for the first joint. This
-         allows accessing different operational areas, e.g. left-handed vs.
-         right-handed robots. -->
-    <crane_plus parent="base_link"
-                servo_color="black" bracket_color="grey" gripper_color="black"
-                joints_vlimit="1.571"
-                pan_llimit="-2.617" pan_ulimit="2.617">
-      <!-- Place the "floating" arm at the location it should be if mounted on
-           a TurtleBot, as pick and place and other demos assume this
-           location -->
-      <!--<origin xyz="0.1 0.03 0.435"/>-->
-      <origin xyz="0 0 0"/>
-    </crane_plus>
+  <!-- Include the Crane+ generator macro -->
+  <xacro:include filename="$(find crane_plus_description)/urdf/crane_plus.xacro"/>
+  <!-- Link to provide the location reference for the arm -->
+  <link name="base_link"/>
+  <!-- Use the crane_plus macro to configure a Crane+ arm with desired joint
+       velocities limit and lower/upper limits for the first joint. This
+       allows accessing different operational areas, e.g. left-handed vs.
+       right-handed robots. -->
+  <crane_plus parent="base_link"
+              servo_color="black" bracket_color="grey" gripper_color="black"
+              joints_vlimit="1.571"
+              pan_llimit="-2.617" pan_ulimit="2.617">
+    <!-- Place the "floating" arm at the location it should be if mounted on
+         a TurtleBot, as pick and place and other demos assume this
+         location -->
+    <!--<origin xyz="0.1 0.03 0.435"/>-->
+    <origin xyz="0 0 0"/>
+  </crane_plus>
 </robot>

File: crane_plus_description/urdf/crane_plus_hardware.xacro (robot description, xacro)
@@ -57,9 +57,9 @@
     <link name="${name}_link">
       <inertial>
-        <mass value="0.00001"/>
-        <origin xyz="0 0 0"/>
-        <inertia ixx="1.0" ixy="0.0" ixz="0.0"
-          iyy="1.0" iyz="0.0"
-          izz="1.0"/>
+        <mass value="0.02"/>
+        <origin xyz="0 0 0.0005" rpy="0 0 0"/>
+        <inertia ixx="4.1683e-6" ixy="0.0" ixz="0.0"
+          iyy="8.33e-6" iyz="0.0"
+          izz="4.1683e-6"/>
       </inertial>
       <visual>
@@ -86,9 +86,9 @@
     <link name="${name}_link">
       <inertial>
-        <mass value="0.00001"/>
-        <origin xyz="0 0 0"/>
-        <inertia ixx="1.0" ixy="0.0" ixz="0.0"
-          iyy="1.0" iyz="0.0"
-          izz="1.0"/>
+        <mass value="0.005"/>
+        <origin xyz="0.0 0.0 0.004" rpy="0 0 0"/>
+        <inertia ixx="4.53e-7" ixy="0.0" ixz="0.0"
+          iyy="6.283e-7" iyz="0.0"
+          izz="2.283e-7"/>
       </inertial>
       <visual>
@@ -115,9 +115,9 @@
     <link name="${name}_link">
       <inertial>
-        <mass value="0.00001"/>
-        <origin xyz="0 0 0"/>
-        <inertia ixx="1.0" ixy="0.0" ixz="0.0"
-          iyy="1.0" iyz="0.0"
-          izz="1.0"/>
+        <mass value="0.0564"/>
+        <origin xyz="${0-AX12_ORIGIN_OFFSET_X} 0 0" rpy="0 0 0"/>
+        <inertia ixx="1.16e-5" ixy="0.0" ixz="0.0"
+          iyy="1.656e-50" iyz="0.0"
+          izz="1.854e-5"/>
       </inertial>
       <visual>
@@ -146,9 +146,9 @@
     <link name="${name}_link">
       <inertial>
-        <mass value="0.00001"/>
-        <origin xyz="0 0 0"/>
-        <inertia ixx="1.0" ixy="0.0" ixz="0.0"
-          iyy="1.0" iyz="0.0"
-          izz="1.0"/>
+        <mass value="0.0564"/>
+        <origin xyz="${AX12_ORIGIN_TO_AXLE-AX12_ORIGIN_OFFSET_X} 0 0" rpy="0 0 0"/>
+        <inertia ixx="1.16e-5" ixy="0.0" ixz="0.0"
+          iyy="1.656e-5" iyz="0.0"
+          izz="1.854e-5"/>
       </inertial>
       <visual>
@@ -169,5 +169,5 @@
   <xacro:macro name="bioloid_f2_revolute_base_axis" params="parent name color llimit ulimit vlimit *origin">
     <joint name="${name}_joint" type="revolute">
-      <insert_block name="origin"/>
+      <xacro:insert_block name="origin"/>
       <axis xyz="0 0 1"/>
       <limit effort="30" velocity="${vlimit}" lower="${llimit}" upper="${ulimit}"/>
@@ -177,9 +177,11 @@
     <link name="${name}_link">
       <inertial>
-        <mass value="0.00001"/>
-        <origin xyz="0 0 0"/>
-        <inertia ixx="1.0" ixy="0.0" ixz="0.0"
-          iyy="1.0" iyz="0.0"
-          izz="1.0"/>
+        <mass value="0.01"/>
+        <origin xyz="0 0 0.01875" rpy="0 0 0"/>
+        <!-- Full height: (3.1320833333333333e-06, 2.481041666666667e-06, 1.6927083333333333e-06) -->
+        <!-- Half height: (2.253177083333333e-06, 2.481041666666667e-06, 8.138020833333333e-07) -->
+        <inertia ixx="2.253e-6" ixy="0.0" ixz="0.0"
+          iyy="2.481e-6" iyz="0.0"
+          izz="8.138e-7"/>
       </inertial>
       <visual>
@@ -200,5 +202,5 @@
   <xacro:macro name="bioloid_f2_revolute" params="parent name color llimit ulimit vlimit *origin">
     <joint name="${name}_joint" type="revolute">
-      <insert_block name="origin"/>
+      <xacro:insert_block name="origin"/>
       <axis xyz="0 1 0"/>
       <limit effort="30" velocity="${vlimit}" lower="${llimit}" upper="${ulimit}"/>
@@ -208,9 +210,11 @@
     <link name="${name}_link">
       <inertial>
-        <mass value="0.00001"/>
-        <origin xyz="0 0 0"/>
-        <inertia ixx="1.0" ixy="0.0" ixz="0.0"
-          iyy="1.0" iyz="0.0"
-          izz="1.0"/>
+        <mass value="0.01"/>
+        <origin xyz="0 0 -${F2_AXLE_HEIGHT-F2_HEIGHT/2}" rpy="0 0 0"/>
+        <!-- Full height: (3.1320833333333333e-06, 2.481041666666667e-06, 1.6927083333333333e-06) -->
+        <!-- Half height: (2.253177083333333e-06, 2.481041666666667e-06, 8.138020833333333e-07) -->
+        <inertia ixx="2.253e-6" ixy="0.0" ixz="0.0"
+          iyy="2.481e-6" iyz="0.0"
+          izz="8.138e-7"/>
       </inertial>
       <visual>
@@ -237,9 +241,9 @@
     <link name="${name}_link">
       <inertial>
-        <mass value="0.00001"/>
-        <origin xyz="0 0 0"/>
-        <inertia ixx="1.0" ixy="0.0" ixz="0.0"
-          iyy="1.0" iyz="0.0"
-          izz="1.0"/>
+        <mass value="0.005"/>
+        <origin xyz="0.0 0.0 0.0045" rpy="0 0 0"/>
+        <inertia ixx="6.354e-7" ixy="0.0" ixz="0.0"
+          iyy="8.621e-7" iyz="0.0"
+          izz="2.942e-7"/>
       </inertial>
       <visual>
@@ -260,5 +264,5 @@
   <xacro:macro name="bioloid_f4_revolute" params="parent name color llimit ulimit vlimit *origin">
     <joint name="${name}_joint" type="revolute">
-      <insert_block name="origin"/>
+      <xacro:insert_block name="origin"/>
       <axis xyz="0 1 0"/>
       <limit effort="30" velocity="${vlimit}" lower="${llimit}" upper="${ulimit}"/>
@@ -268,9 +272,11 @@
     <link name="${name}_link">
       <inertial>
-        <mass value="0.00001"/>
-        <origin xyz="0 0 0"/>
-        <inertia ixx="1.0" ixy="0.0" ixz="0.0"
-          iyy="1.0" iyz="0.0"
-          izz="1.0"/>
+        <mass value="0.015"/>
+        <origin xyz="0 0 -${F4_AXLE_HEIGHT-F4_HEIGHT/2+0.0015}" rpy="0 0 0"/>
+        <!-- Full height: (8.2215625e-06, 3.9203124999999996e-06, 6.2612499999999996e-06) -->
+        <!-- Half height: (4.2606249999999995e-06, 3.9203124999999996e-06, 2.3003125e-06) -->
+        <inertia ixx="4.261e-6" ixy="0.0" ixz="0.0"
+          iyy="3.921e-6" iyz="0.0"
+          izz="2.3e-6"/>
       </inertial>
       <visual>
@@ -299,9 +305,9 @@
     <link name="${name}_link">
       <inertial>
-        <mass value="0.00001"/>
-        <origin xyz="0 0 0"/>
-        <inertia ixx="1.0" ixy="0.0" ixz="0.0"
-          iyy="1.0" iyz="0.0"
-          izz="1.0"/>
+        <mass value="0.02"/>
+        <origin xyz="0 0 0" rpy="0 0 0"/>
+        <inertia ixx="1.612e-5" ixy="0.0" ixz="0.0"
+          iyy="1.823e-5" iyz="0.0"
+          izz="2.732e-6"/>
       </inertial>
       <visual>
@@ -328,9 +334,9 @@
     <link name="${name}_link">
       <inertial>
-        <mass value="0.00001"/>
-        <origin xyz="0 0 0"/>
-        <inertia ixx="1.0" ixy="0.0" ixz="0.0"
-          iyy="1.0" iyz="0.0"
-          izz="1.0"/>
+        <mass value="0.02"/>
+        <origin xyz="0 0 0" rpy="0 0 0"/>
+        <inertia ixx="2.01e-5" ixy="0.0" ixz="0.0"
+          iyy="2.2e-5" iyz="0.0"
+          izz="2.936e-6"/>
       </inertial>
       <visual>

File: crane_plus_simulation/urdf/simulated_crane_plus.urdf (robot description, URDF)
Before this commit: robot crane_plus_arm, 20 links, 19 joints
Links:
- removed link base_link
- added link world
Joints:
- joint crane_plus_base_joint: parent base_link -> world

Commit message: Remove ancient comment

File: crane_plus_description/urdf/crane_plus.urdf.xacro (robot description, xacro)
@@ -18,8 +18,4 @@
               joints_vlimit="1.571"
               pan_llimit="-2.617" pan_ulimit="2.617">
-    <!-- Place the "floating" arm at the location it should be if mounted on
-         a TurtleBot, as pick and place and other demos assume this
-         location -->
-    <!--<origin xyz="0.1 0.03 0.435"/>-->
     <origin xyz="0 0 0"/>
   </crane_plus>
